Commit message: Changed the model to actually be a chain.
Now it starts from base_footprint and it goes up all the way to the neck and arms
in the same way you would find in any other mobile base robot.
This enables standard usage of MoveIt! and other tools as the TF tree
can form a chain.

File: pepper_description/urdf/pepper1.0_generated_urdf/pepper_arms.xacro (robot description, xacro)
@@ -7,5 +7,5 @@
 		<parent link="torso"/>
 		<child link="LShoulder"/>
-		<origin rpy="0 0 0" xyz="-0.057 0.14974 0.08682"/>
+		<origin rpy="0 0 0" xyz="-0.057 0.14974 ${0.08682 + 0.139}"/>
 		<axis xyz="0 1.0 0"/>
 		<limit effort="5.428" lower="-2.08567" upper="2.08567" velocity="7.33998"/>
@@ -95,5 +95,5 @@
 		<parent link="torso"/>
 		<child link="RShoulder"/>
-		<origin rpy="0 0 0" xyz="-0.057 -0.14974 0.08682"/>
+		<origin rpy="0 0 0" xyz="-0.057 -0.14974 ${0.08682 + 0.139}"/>
 		<axis xyz="0 1.0 0"/>
 		<limit effort="5.428" lower="-2.08567" upper="2.08567" velocity="7.33998"/>

File: pepper_description/urdf/pepper1.0_generated_urdf/pepper_head.xacro (robot description, xacro)
@@ -7,5 +7,5 @@
 		<parent link="torso"/>
 		<child link="Neck"/>
-		<origin rpy="0 0 0" xyz="-0.038 0 0.1699"/>
+		<origin rpy="0 0 0" xyz="-0.038 0 ${0.1699 + 0.139}"/>
 		<axis xyz="0 0 1.0"/>
 		<limit effort="5.428" lower="-2.08567" upper="2.08567" velocity="7.33998"/>

File: pepper_description/urdf/pepper1.0_generated_urdf/pepper_legs.xacro (robot description, xacro)
@@ -5,7 +5,7 @@
 <robot xmlns:xacro="http://www.ros.org/wiki/xacro">
 	<joint name="HipRoll" type="revolute">
-		<parent link="torso"/>
-		<child link="Hip"/>
-		<origin rpy="0 0 0" xyz="2e-05 0 -0.139"/>
+		<parent link="Hip"/>
+		<child link="torso"/>
+		<origin rpy="0 0 0" xyz="0 0 0.079"/>
 		<axis xyz="1.0 0 0"/>
 		<limit effort="10.1884" lower="-0.514872" upper="0.514872" velocity="2.27032"/>
@@ -20,7 +20,7 @@
 	</link>
 	<joint name="HipPitch" type="revolute">
-		<parent link="Hip"/>
-		<child link="Pelvis"/>
-		<origin rpy="0 0 0" xyz="0 0 -0.079"/>
+		<parent link="Pelvis"/>
+		<child link="Hip"/>
+		<origin rpy="0 0 0" xyz="0 0 0.268"/>
 		<axis xyz="0 1.0 0"/>
 		<limit effort="19.787" lower="-1.03847" upper="1.03847" velocity="2.93276"/>
@@ -35,7 +35,7 @@
 	</link>
 	<joint name="KneePitch" type="revolute">
-		<parent link="Pelvis"/>
-		<child link="Tibia"/>
-		<origin rpy="0 0 0" xyz="0 0 -0.268"/>
+		<parent link="Tibia"/>
+		<child link="Pelvis"/>
+		<origin rpy="0 0 0" xyz="0 0 0"/>
 		<axis xyz="0 1.0 0"/>
 		<limit effort="27.702" lower="-0.514872" upper="0.514872" velocity="2.93276"/>
@@ -50,7 +50,7 @@
 	</link>
 	<joint name="base_footprint_joint" type="fixed">
-		<parent link="Tibia"/>
-		<child link="base_footprint"/>
-		<origin rpy="0 0 0" xyz="0 0 -0.334"/>
+		<parent link="base_footprint"/>
+		<child link="Tibia"/>
+		<origin rpy="0 0 0" xyz="0 0 0.334"/>
 	</joint>
 	<link name="base_footprint"/>

File: pepper_description/urdf/pepper1.0_generated_urdf/pepper_torso.xacro (robot description, xacro)
@@ -6,6 +6,6 @@
 	<link name="base_link"/>
 	<joint name="base_link_fixedjoint" type="fixed">
-		<parent link="base_link"/>
-		<child link="torso"/>
+		<parent link="torso"/>
+		<child link="base_link"/>
 		<origin rpy="0 0 0" xyz="0 0 0"/>
 		<axis xyz="0 0 0"/>

File: pepper_description/urdf/pepper1.0_generated_urdf/pepper_visual_collisions.xacro (robot description, xacro)
@@ -35,11 +35,11 @@
 		<visual>
 			<geometry>
-				<mesh filename="package://pepper_meshes/meshes/1.0/HipRoll.dae" scale="0.1 0.1 0.1"/>
-			</geometry>
-			<origin rpy="0 0 0" xyz="0 0 0"/>
-		</visual>
-		<collision>
-			<geometry>
-				<mesh filename="package://pepper_meshes/meshes/1.0/HipRoll_0.10.stl" scale="0.1 0.1 0.1"/>
+				<mesh filename="package://pepper_description/meshes/HipRoll.dae" scale="0.1 0.1 0.1"/>
+			</geometry>
+			<origin rpy="0 0 0" xyz="0 0 0"/>
+		</visual>
+		<collision>
+			<geometry>
+				<mesh filename="package://pepper_description/meshes/HipRoll_0.10.stl" scale="0.1 0.1 0.1"/>
 			</geometry>
 			<origin rpy="0 0 0" xyz="0 0 0"/>
@@ -539,11 +539,11 @@
 		<visual>
 			<geometry>
-				<mesh filename="package://pepper_meshes/meshes/1.0/Torso.dae" scale="0.1 0.1 0.1"/>
-			</geometry>
-			<origin rpy="0 0 0" xyz="0 0 0"/>
-		</visual>
-		<collision>
-			<geometry>
-				<mesh filename="package://pepper_meshes/meshes/1.0/Torso_0.10.stl" scale="0.1 0.1 0.1"/>
+				<mesh filename="package://pepper_description/meshes/Torso.dae" scale="0.1 0.1 0.1"/>
+			</geometry>
+			<origin rpy="0 0 0" xyz="0 0 0"/>
+		</visual>
+		<collision>
+			<geometry>
+				<mesh filename="package://pepper_description/meshes/Torso_0.10.stl" scale="0.1 0.1 0.1"/>
 			</geometry>
 			<origin rpy="0 0 0" xyz="0 0 0"/>
@@ -651,11 +651,11 @@
 		<visual>
 			<geometry>
-				<mesh filename="package://pepper_meshes/meshes/1.0/HipPitch.dae" scale="0.1 0.1 0.1"/>
-			</geometry>
-			<origin rpy="0 0 0" xyz="0 0 0"/>
-		</visual>
-		<collision>
-			<geometry>
-				<mesh filename="package://pepper_meshes/meshes/1.0/HipPitch_0.10.stl" scale="0.1 0.1 0.1"/>
+				<mesh filename="package://pepper_description/meshes/HipPitch.dae" scale="0.1 0.1 0.1"/>
+			</geometry>
+			<origin rpy="0 0 0" xyz="0 0 0"/>
+		</visual>
+		<collision>
+			<geometry>
+				<mesh filename="package://pepper_description/meshes/HipPitch_0.10.stl" scale="0.1 0.1 0.1"/>
 			</geometry>
 			<origin rpy="0 0 0" xyz="0 0 0"/>
