Commit message: Fixed joint directions.
This was a terrible bug that made the joints twist in the inverse direction so every time
the robot wasnt in a standing position the transforms were wrong

File: pepper_description/urdf/pepper1.0_generated_urdf/pepper_legs.xacro (robot description, xacro)
@@ -8,5 +8,5 @@
 		<child link="torso"/>
 		<origin rpy="0 0 0" xyz="0 0 0.079"/>
-		<axis xyz="1.0 0 0"/>
+		<axis xyz="-1.0 0 0"/>
 		<limit effort="10.1884" lower="-0.514872" upper="0.514872" velocity="2.27032"/>
 	</joint>
@@ -23,5 +23,5 @@
 		<child link="Hip"/>
 		<origin rpy="0 0 0" xyz="0 0 0.268"/>
-		<axis xyz="0 1.0 0"/>
+		<axis xyz="0 -1.0 0"/>
 		<limit effort="19.787" lower="-1.03847" upper="1.03847" velocity="2.93276"/>
 	</joint>
@@ -38,5 +38,5 @@
 		<child link="Pelvis"/>
 		<origin rpy="0 0 0" xyz="0 0 0"/>
-		<axis xyz="0 1.0 0"/>
+		<axis xyz="0 -1.0 0"/>
 		<limit effort="27.702" lower="-0.514872" upper="0.514872" velocity="2.93276"/>
 	</joint>
