Commit message: Added missing files because of branch error

File: pepper_description/urdf/pepper1.0_generated_urdf/pepperTransmission_no_arms.xacro (robot description, xacro)
@@ -87,6 +87,6 @@
 		</transmission> -->
 		</xacro:macro>
-	<xacro:arm_joints_transmissions side="L"/>
-	<xacro:arm_joints_transmissions side="R"/>
+	<!-- <xacro:arm_joints_transmissions side="L"/>
+	<xacro:arm_joints_transmissions side="R"/> -->
 	<!-- LEGS -->
 	<transmission name="HipRoll_Transmission">

File: pepper_description/urdf/pepper1.0_generated_urdf/pepper_legs.xacro (robot description, xacro)
@@ -43,6 +43,8 @@
 	<link name="Tibia">
 		<inertial>
-			<mass value="11.6015"/>
-			<inertia ixx="0.129229" ixy="-0.000401943" ixz="0.00048556" iyy="0.122839" iyz="-1.01666e-08" izz="0.108168"/>
+			<!-- We increase the weight of the base and nullify anything but the diagonal on the inertia matrix
+			to help the plugins that move the base to not slip in weird ways -->
+			<mass value="${11.6015 * 100.0}"/>
+			<inertia ixx="${0.129229 * 100.0}" ixy="${-0.000401943 * 0.0}" ixz="${0.00048556 * 0.0}" iyy="${0.122839 * 100.0}" iyz="${-1.01666e-08 * 0.0}" izz="${0.108168 * 100.0}"/>
 			<origin rpy="0 0 0" xyz="0.00220451 0 -0.185729"/>
 		</inertial>

File: pepper_description/urdf/pepper1.0_generated_urdf/pepper_robot_CPU.xacro (robot description, xacro)
@@ -12,5 +12,5 @@
 	<!-- <xacro:include filename="pepper_fingers.xacro"/> -->
 	<xacro:include filename="pepper_wheels.xacro"/>
-	<xacro:include filename="pepperGazebo.xacro"/>
+	<xacro:include filename="pepperGazeboCPU.xacro"/>
 	<xacro:include filename="pepperTransmission.xacro"/>
 </robot>

File: pepper_description/urdf/pepper1.0_generated_urdf/pepper_robot_CPU_no_arms.xacro (robot description, xacro)
@@ -8,9 +8,9 @@
 	<xacro:include filename="pepper_legs.xacro"/>
 	<xacro:include filename="pepper_torso.xacro"/>
-	<xacro:include filename="pepper_arms.xacro"/>
-	<xacro:include filename="pepper_sensors.xacro"/>
+	<!-- <xacro:include filename="pepper_arms.xacro"/> -->
+	<xacro:include filename="pepper_sensors_no_arms.xacro"/>
 	<!-- <xacro:include filename="pepper_fingers.xacro"/> -->
 	<xacro:include filename="pepper_wheels.xacro"/>
-	<xacro:include filename="pepperGazebo.xacro"/>
-	<xacro:include filename="pepperTransmission.xacro"/>
+	<xacro:include filename="pepperGazeboCPU_no_arms.xacro"/>
+	<xacro:include filename="pepperTransmission_no_arms.xacro"/>
 </robot>

File: pepper_description/urdf/pepper1.0_generated_urdf/pepper_sensors_no_arms.xacro (robot description, xacro)
@@ -23,5 +23,5 @@
 		<origin rpy="-1.57079632679 0 -1.57079632679" xyz="0 0 0"/>
 	</joint>
-	<link name="LHandTouchBack_frame"/>
+<!-- 	<link name="LHandTouchBack_frame"/>
 	<joint name="LHand/Touch/Back_sensor_fixedjoint" type="fixed">
 		<parent link="l_wrist"/>
@@ -29,5 +29,5 @@
 		<origin rpy="1.5708 -1.5708 -3.14159" xyz="0.0523 0 0.0304"/>
 		<axis xyz="0 0 0"/>
-	</joint>
+	</joint> -->
 	<link name="VerticalLeftLaser_frame"/>
 	<joint name="LaserSensor/VerticalLeft_sensor_fixedjoint" type="fixed">
@@ -93,5 +93,5 @@
 		<axis xyz="0 0 0"/>
 	</joint>
-	<link name="RHandTouchBack_frame"/>
+<!-- 	<link name="RHandTouchBack_frame"/>
 	<joint name="RHand/Touch/Back_sensor_fixedjoint" type="fixed">
 		<parent link="r_wrist"/>
@@ -99,5 +99,5 @@
 		<origin rpy="1.5708 -1.5708 -3.14159" xyz="0.0523 0 0.0304"/>
 		<axis xyz="0 0 0"/>
-	</joint>
+	</joint> -->
 	<link name="CameraTop_frame"/>
 	<joint name="CameraTop_sensor_fixedjoint" type="fixed">

File: pepper_description/urdf/pepper1.0_generated_urdf/pepper_visual_collisions.xacro (robot description, xacro)
@@ -109,10 +109,10 @@
 			<origin rpy="0 0 0" xyz="0 0 0"/>
 		</visual>
-		<collision>
+<!-- 		<collision>
 			<geometry>
 				<mesh filename="package://pepper_meshes/meshes/1.0/WheelFL_0.10.stl" scale="0.1 0.1 0.1"/>
 			</geometry>
 			<origin rpy="0 0 0" xyz="0 0 0"/>
-		</collision>
+		</collision> -->
 	</xacro:macro>
 	<xacro:macro name="insert_visu_LFinger21_link">
@@ -251,7 +251,11 @@
 		<collision>
 			<geometry>
-				<mesh filename="package://pepper_meshes/meshes/1.0/KneePitch_0.10.stl" scale="0.1 0.1 0.1"/>
-			</geometry>
-			<origin rpy="0 0 0" xyz="0 0 0"/>
+<!-- 				<mesh filename="package://pepper_meshes/meshes/1.0/KneePitch_0.10.stl" scale="0.1 0.1 0.1"/>
+ -->
+                <!-- We approximate the base with a box to ease the contacts with the ground so
+                plugins that move the base actually work -->
+ 				<box size="0.35 0.35 0.2"/>
+ 			</geometry>
+			<origin rpy="0 0 0" xyz="0 0 ${-0.24}"/>
 		</collision>
 	</xacro:macro>
@@ -459,10 +463,10 @@
 			<origin rpy="0 0 0" xyz="0 0 0"/>
 		</visual>
-		<collision>
+<!-- 		<collision>
 			<geometry>
 				<mesh filename="package://pepper_meshes/meshes/1.0/WheelB_0.10.stl" scale="0.1 0.1 0.1"/>
 			</geometry>
 			<origin rpy="0 0 0" xyz="0 0 0"/>
-		</collision>
+		</collision> -->
 	</xacro:macro>
 	<xacro:macro name="insert_visu_LFinger23_link">
@@ -627,10 +631,10 @@
 			<origin rpy="0 0 0" xyz="0 0 0"/>
 		</visual>
-		<collision>
+<!-- 		<collision>
 			<geometry>
 				<mesh filename="package://pepper_meshes/meshes/1.0/WheelFR_0.10.stl" scale="0.1 0.1 0.1"/>
 			</geometry>
 			<origin rpy="0 0 0" xyz="0 0 0"/>
-		</collision>
+		</collision> -->
 	</xacro:macro>
 	<xacro:macro name="insert_visu_LShoulder">
